File: Interboard_connector.kicad_sch (KiCad schematic)
At the start: 2 parts, among them J1 Chainbus in, J2 Chainbus Out

Commit message: changed vin connector to hierarchical labels
Connections:
- net BRD_VIN renamed VIN_CHAINBUS
