File: Bus_switch.kicad_sch (KiCad schematic)
At the start: 15 parts, among them J3 Conn_01x04_Pin, U1 SN74CB3Q3384APW

Commit message: fixed selected led polarity
Connections:
- net +3V3: now also D3.2
- net GND: no longer D3.1
- net at R1.2: now also D3.1; no longer D3.2
