File: MMS3_hat_templates.kicad_pcb (KiCad board)
At the start: 2 copper layers, 100 x 50 mm, 35 parts, among them J1 Chainbus in, J2 Chainbus Out, J3 Conn_01x04_Pin, J4 AMASS XT60 Male, J5 AMASS XT60 Female, U1 SN74CB3Q3384APW, U2 M24C64, U4 AMS1117

Commit message: added missing 3D models for XT60
Other:
- board text removed: "J1"
- board text removed: "J2"
- board text removed: "SN74CB3Q3384APW"
- board text removed: "TMC5130A-TA"
- board text removed: "U1"
