File: MMS3_hat_templates.kicad_pcb (KiCad board)
At the start: 2 copper layers, 100 x 50 mm, 35 parts, among them J1 Chainbus in, J2 Chainbus Out, J3 Conn_01x04_Pin, J4 AMASS XT60 Male, J5 AMASS XT60 Female, U1 SN74CB3Q3384APW, U2 M24C64, U4 AMS1117

Commit message: added box around chainbus bus switch in schematic
Parts:
- removed R11, R2, R3, R5, R7, R8, R9: 10kΩ, PCM_JLCPCB:R_0402
Routing:
- net +12V stby: track 2.34 -> 4.68 mm, vias 1 -> 2
