File: Hardware/Interboard_connector.kicad_sch (KiCad schematic)
At the start: 2 parts, among them J1 Chainbus in, J2 Chainbus Out

Commit message: removed holes from bom
Other:
- company: Moducard System -> MiniModucard System
Changed lines of the file:
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@@
 	(title_block
 		(title "MMS3 Hat template small (Change Me)")
-		(date "2026-02-25")
+		(date "2077-13-75")
 		(rev "A")
-		(company "Moducard System")
-		(comment 1 "Made by Wojciech Szafrański")
+		(company "MiniModucard System")
+		(comment 1 "Wojciech Szafrański")
 		(comment 2 "Designed in poland")
 	)

Commit message: changed numbering to per-sheet
Parts:
- renumbered J1 to J201, J2 to J202

Commit message: MAJOR CHANGE - Pins 25 27 of chainbus connected
Connections:
- net Pin_25: now reaches J202.25 (Pin_25)
- net Pin_25: now also J201.25 (Pin_25)
- net Pin_27: now reaches J202.27 (Pin_27)
- net Pin_27: now also J201.27 (Pin_27)
- no-connect marks 5 -> 1
Changed lines of the file:
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@@
-	)
-	(no_connect
-		(at 113.03 53.34)
-	)
-	(no_connect
-		(at 115.57 53.34)
 	)
 	(no_connect
 		(at 176.53 66.04)
 	)
-	(no_connect
-		(at 191.77 53.34)
-	)
-	(no_connect
-		(at 189.23 53.34)
-	)
 	(bus_entry
 		(at 110.49 85.09)
@@
 	(wire
 		(pts
+			(xy 191.77 43.18) (xy 191.77 53.34)
+		)
+		(stroke
+			(width 0)
+			(type default)
+		)
+	)
+	(wire
+		(pts
 			(xy 90.17 50.8) (xy 90.17 53.34)
 		)
@@
 		)
 	)
+	(wire
+		(pts
+			(xy 113.03 43.18) (xy 113.03 53.34)
+		)
+		(stroke
+			(width 0)
+			(type default)
+		)
+	)
 	(bus
 		(pts
@@
 	(wire
 		(pts
+			(xy 189.23 43.18) (xy 189.23 53.34)
+		)
+		(stroke
+			(width 0)
+			(type default)
+		)
+	)
+	(wire
+		(pts
 			(xy 82.55 66.04) (xy 82.55 67.31)
+		)
+		(stroke
+			(width 0)
+			(type default)
+		)
+	)
+	(wire
+		(pts
+			(xy 115.57 43.18) (xy 115.57 53.34)
 		)
 		(stroke
@@
 		)
 	)
+	(label "Pin_25"
+		(at 189.23 43.18 90)
+		(effects
+			(font
+				(size 1.27 1.27)
+			)
+			(justify left bottom)
+		)
+	)
 	(label "Chainbus.SDA"
 		(at 102.87 67.31 270)
@@
 		)
 	)
+	(label "Pin_25"
+		(at 113.03 43.18 90)
+		(effects
+			(font
+				(size 1.27 1.27)
+			)
+			(justify left bottom)
+		)
+	)
 	(label "SEL6"
 		(at 95.25 76.2 270)
@@
 		)
 	)
+	(label "Pin_27"
+		(at 115.57 43.18 90)
+		(effects
+			(font
+				(size 1.27 1.27)
+			)
+			(justify left bottom)
+		)
+	)
 	(label "Chainbus.RX"
 		(at 196.85 67.31 270)
@@
 		)
 	)
+	(label "Pin_27"
+		(at 191.77 43.18 90)
+		(effects
+			(font
+				(size 1.27 1.27)
+			)
+			(justify left bottom)
+		)
+	)
