File: Hardware/Interboard_connector.kicad_sch (KiCad schematic)
At the start: 2 parts, among them J201 Chainbus in, J202 Chainbus Out

Commit message: added UART flip information
Other:
- note added: "UART FLIP"

Commit message: major rework of template
Other:
- note added: "UART FLIP STATUS"
- note removed: "UART FLIP"
Changed lines of the file:
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@@
 		)
 	)
-	(text "UART FLIP"
+	(text "UART FLIP STATUS"
 		(exclude_from_sim no)
 		(at 26.67 190.5 0)

Commit message: added LCSC numbers to chainbus connectors
Parts:
- J201: LCSC (none) -> C6332241
- J202: LCSC (none) -> C41380407
Changed lines of the file:
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@@
+			)
+		)
+		(property "LCSC" "C41380407"
+			(at 140.97 64.77 90)
+			(hide yes)
+			(show_name no)
+			(do_not_autoplace no)
+			(effects
+				(font
+					(size 1.27 1.27)
+				)
 			)
 		)
@@
 			(at 64.77 64.77 90)
 			(hide yes)
+			(show_name no)
+			(do_not_autoplace no)
+			(effects
+				(font
+					(size 1.27 1.27)
+				)
+			)
+		)
+		(property "LCSC" "C6332241"
+			(at 64.77 64.77 90)
+			(hide yes)
