File: Hardware/MMS3_hat_templates.kicad_sch (KiCad schematic)
At the start: 12 parts, among them U4 AMS1117

Commit message: removed holes from bom
Parts:
- removed H7, H8, H9: (no value), PCM_JLCPCB:Hole_Tooling_JLCPCB, symbol PCM_JLCPCB-Manufacturing:Tooling Hole, PCM_JLCPCB, 1.152mm
- H1, H2, H3, H4, H5, H6: now not fitted

Commit message: changed numbering to per-sheet
Parts:
- renumbered C16 to C101, C18 to C102, H1 to H101, H2 to H102, H3 to H103, H4 to H104, H5 to H105, H6 to H106, U4 to U101
Changed lines of the file:
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@@
 		(in_pos_files yes)
 		(dnp no)
-		(property "Reference" "#PWR069"
+		(property "Reference" "#PWR0103"
 			(at 86.36 176.53 0)
 			(hide yes)
@@
 			(project "MMS3_hat_templates"
 				(path "/6596548a-44e0-46d8-8624-fd71cf4a3e17"
-					(reference "#PWR069")
+					(reference "#PWR0103")
 					(unit 1)
 				)
@@
 		(dnp no)
 		(fields_autoplaced yes)
-		(property "Reference" "#SYM2"
+		(property "Reference" "#SYM102"
 			(at 52.07 190.5 90)
 			(hide yes)
@@
 			(project "MMS3_hat_templates"
 				(path "/6596548a-44e0-46d8-8624-fd71cf4a3e17"
-					(reference "#SYM2")
+					(reference "#SYM102")
 					(unit 1)
 				)
@@
 		(dnp no)
 		(fields_autoplaced yes)
-		(property "Reference" "#PWR080"
+		(property "Reference" "#PWR0108"
 			(at 167.64 184.15 0)
 			(hide yes)
@@
 			(project "MMS3_hat_templates"
 				(path "/6596548a-44e0-46d8-8624-fd71cf4a3e17"
-					(reference "#PWR080")
+					(reference "#PWR0108")
 					(unit 1)
 				)
@@
 		(dnp yes)
 		(fields_autoplaced yes)
-		(property "Reference" "H2"
+		(property "Reference" "H102"
 			(at 35.56 171.4499 0)
 			(show_name no)
@@
 			(project "MMS3_hat_templates"
 				(path "/6596548a-44e0-46d8-8624-fd71cf4a3e17"
-					(reference "H2")
+					(reference "H102")
 					(unit 1)
 				)
@@
 		(dnp no)
 		(fields_autoplaced yes)
-		(property "Reference" "#FLG01"
+		(property "Reference" "#FLG0101"
 			(at 157.48 179.705 0)
 			(hide yes)
@@
 			(project "MMS3_hat_templates"
 				(path "/6596548a-44e0-46d8-8624-fd71cf4a3e17"
-					(reference "#FLG01")
+					(reference "#FLG0101")
 					(unit 1)
 				)
@@
 		(dnp no)
 		(fields_autoplaced yes)
-		(property "Reference" "#PWR073"
+		(property "Reference" "#PWR0105"
 			(at 110.49 195.58 0)
 			(hide yes)
@@
 			(project "MMS3_hat_templates"
 				(path "/6596548a-44e0-46d8-8624-fd71cf4a3e17"
-					(reference "#PWR073")
+					(reference "#PWR0105")
 					(unit 1)
 				)
@@
 		(dnp no)
 		(fields_autoplaced yes)
-		(property "Reference" "#PWR075"
+		(property "Reference" "#PWR0106"
 			(at 127 195.58 0)
 			(hide yes)
@@
 			(project "MMS3_hat_templates"
 				(path "/6596548a-44e0-46d8-8624-fd71cf4a3e17"
-					(reference "#PWR075")
+					(reference "#PWR0106")
 					(unit 1)
 				)
@@
 		(dnp yes)
 		(fields_autoplaced yes)
-		(property "Reference" "H3"
+		(property "Reference" "H103"
 			(at 35.56 176.5299 0)
 			(show_name no)
@@
 			(project "MMS3_hat_templates"
 				(path "/6596548a-44e0-46d8-8624-fd71cf4a3e17"
-					(reference "H3")
+					(reference "H103")
 					(unit 1)
 				)
@@
 		(dnp no)
 		(fields_autoplaced yes)
-		(property "Reference" "#PWR01"
+		(property "Reference" "#PWR0101"
 			(at 16.51 186.69 0)
 			(hide yes)
@@
 			(project "MMS3_hat_templates"
 				(path "/6596548a-44e0-46d8-8624-fd71cf4a3e17"
-					(reference "#PWR01")
+					(reference "#PWR0101")
 					(unit 1)
 				)
@@
 		(dnp no)
 		(fields_autoplaced yes)
-		(property "Reference" "C18"
+		(property "Reference" "C102"
 			(at 129.54 179.0699 0)
 			(show_name no)
@@
 			(project "MMS3_hat_templates"
 				(path "/6596548a-44e0-46d8-8624-fd71cf4a3e17"
-					(reference "C18")
+					(reference "C102")
 					(unit 1)
 				)
@@
 		(dnp no)
 		(fields_autoplaced yes)
-		(property "Reference" "#SYM1"
+		(property "Reference" "#SYM101"
 			(at 55.88 178.054 0)
 			(hide yes)
@@
 			(project "MMS3_hat_templates"
 				(path "/6596548a-44e0-46d8-8624-fd71cf4a3e17"
-					(reference "#SYM1")
+					(reference "#SYM101")
 					(unit 1)
 				)
@@
 		(dnp yes)
 		(fields_autoplaced yes)
-		(property "Reference" "H4"
+		(property "Reference" "H104"
 			(at 35.56 181.6099 0)
 			(show_name no)
@@
 			(project "MMS3_hat_templates"
 				(path "/6596548a-44e0-46d8-8624-fd71cf4a3e17"
-					(reference "H4")
+					(reference "H104")
 					(unit 1)
 				)
@@
 		(dnp yes)
 		(fields_autoplaced yes)
-		(property "Reference" "H1"
+		(property "Reference" "H101"
 			(at 19.05 171.4499 0)
 			(show_name no)
@@
 			(project "MMS3_hat_templates"
 				(path "/6596548a-44e0-46d8-8624-fd71cf4a3e17"
-					(reference "H1")
+					(reference "H101")
 					(unit 1)
 				)
@@
 		(dnp no)
 		(fields_autoplaced yes)
-		(property "Reference" "U4"
+		(property "Reference" "U101"
 			(at 110.49 168.91 0)
 			(show_name no)
@@
 			(project "MMS3_hat_templates"
 				(path "/6596548a-44e0-46d8-8624-fd71cf4a3e17"
-					(reference "U4")
+					(reference "U101")
 					(unit 1)
 				)
@@
 		(dnp yes)
 		(fields_autoplaced yes)
-		(property "Reference" "H5"
+		(property "Reference" "H105"
 			(at 35.56 186.6899 0)
 			(show_name no)
@@
 			(project "MMS3_hat_templates"
 				(path "/6596548a-44e0-46d8-8624-fd71cf4a3e17"
-					(reference "H5")
+					(reference "H105")
 					(unit 1)
 				)
@@
 		(dnp no)
 		(fields_autoplaced yes)
-		(property "Reference" "C16"
+		(property "Reference" "C101"
 			(at 95.25 180.3399 0)
 			(show_name no)
@@
 			(project "MMS3_hat_templates"
 				(path "/6596548a-44e0-46d8-8624-fd71cf4a3e17"
-					(reference "C16")
+					(reference "C101")
 					(unit 1)
 				)
@@
 		(in_pos_files yes)
 		(dnp no)
-		(property "Reference" "#PWR055"
+		(property "Reference" "#PWR0102"
 			(at 50.8 140.97 0)
 			(hide yes)
@@
 			(project "MMS3_hat_templates"
 				(path "/6596548a-44e0-46d8-8624-fd71cf4a3e17"
-					(reference "#PWR055")
+					(reference "#PWR0102")
 					(unit 1)
 				)
@@
 		(dnp yes)
 		(fields_autoplaced yes)
-		(property "Reference" "H6"
+		(property "Reference" "H106"
 			(at 35.56 191.7699 0)
 			(show_name no)
@@
 			(project "MMS3_hat_templates"
 				(path "/6596548a-44e0-46d8-8624-fd71cf4a3e17"
-					(reference "H6")
+					(reference "H106")
 					(unit 1)
 				)
@@
 		(dnp no)
 		(fields_autoplaced yes)
-		(property "Reference" "#PWR077"
+		(property "Reference" "#PWR0107"
 			(at 132.08 176.53 0)
 			(hide yes)
@@
 			(project "MMS3_hat_templates"
 				(path "/6596548a-44e0-46d8-8624-fd71cf4a3e17"
-					(reference "#PWR077")
+					(reference "#PWR0107")
 					(unit 1)
 				)
@@
 		(dnp no)
 		(fields_autoplaced yes)
-		(property "Reference" "#PWR070"
+		(property "Reference" "#PWR0104"
 			(at 92.71 195.58 0)
 			(hide yes)
@@
 			(project "MMS3_hat_templates"
 				(path "/6596548a-44e0-46d8-8624-fd71cf4a3e17"
-					(reference "#PWR070")
+					(reference "#PWR0104")
 					(unit 1)
 				)

Commit message: major rework of template
Parts:
- added D101: Red, PCM_JLCPCB:D_0603, symbol PCM_JLCPCB-Diodes:LED,0603,Red
- added R101: 1kΩ, PCM_JLCPCB:R_0603, symbol PCM_JLCPCB-Resistors:0603,1kΩ
Connections:
- net +3V3: now also R101.1
- net GND: now also D101.1
- new net: D101.2, R101.2
Other:
- added sheet User Area (User_area.kicad_sch)
- note added: "USER AREA"
- note removed: "<-- Use those connections"
- note removed: "Chainbus connector and bus switch - Do Not Modify"
- moved on the sheet: C101, C102, H101, U101
