File: Hardware/MMS3_hat_templates.kicad_pcb (KiCad board)
At the start: 2 copper layers, 100 x 50 mm, 25 parts, among them J201 Chainbus in, J202 Chainbus Out, J301 Conn_01x04_Pin, J401 AMASS XT60 Male, J402 AMASS XT60 Female, U101 AMS1117, U301 SN74CB3Q3384APW, U501 M24C64

Commit message: major rework of template
Parts:
- removed J401: AMASS XT60 Male, XT60:AMASS_XT60PW-M_1x02_P7.20mm_Horizontal
- removed J402: AMASS XT60 Female, XT60:AMASS_XT60PW-F_1x02_P7.20mm_Horizontal
- removed U301: SN74CB3Q3384APW, Package_SO:TSSOP-24_4.4x7.8mm_P0.65mm
- added CN401: XT60PW-M, lcsc_footprints:C98732_CONN-TH_XT60PW-M, F.Cu at (95.2, 130.7)
- added D101: Red, PCM_JLCPCB:D_0603, F.Cu at (162.9, 103.0)
- added R101: 1kΩ, PCM_JLCPCB:R_0603, F.Cu at (159.8, 103.0)
- added R312: 0Ω, PCM_JLCPCB:R_0603, F.Cu at (144.1, 112.1)
- added R313: 0Ω, PCM_JLCPCB:R_0603, F.Cu at (142.4, 112.1)
- added U302: SN74CB3Q3245PWR, lcsc_footprints:C470961_TSSOP-20_L6_5-W4_4-P0_65-LS6_4-BL, F.Cu at (141.3, 106.6)
- added U401: XT60PW-F_C428722, lcsc_footprints:C428722_TH_2P-XT60PW-F, F.Cu at (111.9, 130.7)
- moved D401 31.0 mm to (83.5, 125.7), turned to -90 degrees
- moved R304 12.9 mm to (166.6, 106.1), turned to -90 degrees
- moved R308 12.3 mm to (165.4, 106.1), turned to -90 degrees
- moved R310 7.56 mm to (147.5, 108.6), turned to 90 degrees
- moved C301 5.82 mm to (145.3, 108.6)
Routing:
- net VIN_CHAINBUS: track 33.7 -> 65.9 mm
- net /Power Connector/VIN_BRD: track 32.9 -> 8.10 mm
- net /Bus_switch/Chainbus.SCL: track 36.0 -> 53.2 mm
- net +3V3: track 57.9 -> 74.7 mm, vias 4 -> 5
- net /Bus_switch/Chainbus.SDA: track 39.7 -> 51.8 mm, vias 2 -> 0
- net /Bus_switch/Chainbus_In.SDA: track 20.4 -> 12.0 mm, vias 2 -> 1
- net /Bus_switch/Chainbus_In.SCL: track 18.6 -> 10.6 mm, vias 2 -> 1
- net /Bus_switch/SEL1: track 82.7 -> 89.7 mm, vias 4 -> 1
- net /Bus_switch/Chainbus_In.CS: track 14.2 -> 8.51 mm
- net /Bus_switch/Chainbus_In.RX: track 5.78 -> 9.96 mm
- net /Bus_switch/Poka_Yoke_RX: track 0.00 -> 3.93 mm
- net /Bus_switch/Chainbus_In.TX: track 6.24 -> 8.13 mm
- net /Bus_switch/Poka_Yoke_TX: track 0.00 -> 1.88 mm
- net Net-(D101-Pad2): track 0.00 -> 1.44 mm
- net /Bus_switch/Chainbus_In.MOSI: track 7.79 -> 6.40 mm
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- added copper zone on B.Cu, net /Power Connector/VIN_BRD
Other:
- board text removed: "DIN41612"

Commit message: improve layout
Parts:
- moved D401 4.96 mm to (83.7, 130.7), turned to 0 degrees
- moved R310 3.65 mm to (145.3, 105.7)
- moved R308 2.13 mm to (167.0, 107.5)
- moved R304 1.65 mm to (167.0, 104.5)
- moved R312 0.76 mm to (143.8, 112.8)
- moved R313 0.76 mm to (142.1, 112.8)
Routing:
- net VIN_CHAINBUS: track 65.9 -> 83.5 mm
- net GND: track 17.5 -> 4.04 mm, vias 25 -> 30
- net +3V3: track 74.7 -> 81.8 mm, vias 5 -> 6
- net /Bus_switch/Chainbus.SCL: track 53.2 -> 48.6 mm, vias 0 -> 2
- net /Bus_switch/SEL1: track 89.7 -> 85.4 mm
- net /Bus_switch/Chainbus.SDA: track 51.8 -> 47.6 mm, vias 0 -> 2
- net +5V: track 58.4 -> 55.0 mm
- net /Bus_switch/Chainbus_In.RX: track 9.96 -> 11.4 mm
- net /Bus_switch/Chainbus_In.TX: track 8.13 -> 9.47 mm
- net /Power Connector/VIN_BRD: track 8.10 -> 7.06 mm
- net /Bus_switch/Chainbus_In.SCK: track 7.02 -> 7.89 mm
- net /Bus_switch/Chainbus_In.SDA: track 12.0 -> 12.8 mm
- net /Bus_switch/Chainbus_In.CS: track 8.51 -> 9.27 mm
- net /Bus_switch/Poka_Yoke_TX: track 1.88 -> 2.47 mm
- net /Bus_switch/Poka_Yoke_RX: track 3.93 -> 4.47 mm
- added copper zone on B.Cu, net +3V3
