File: Hardware/ID_EEPROM.kicad_sch (KiCad schematic)
At the start: 2 parts, among them U2 M24C64

Commit message: removed holes from bom
Other:
- company: (none) -> MiniModucard System
Changed lines of the file:
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@@
 	(title_block
 		(title "MMS3 Hat template small (Change Me)")
-		(date "2026-02-25")
+		(date "2077-13-75")
 		(rev "A")
-		(comment 1 "Made by Wojciech Szafrański")
+		(company "MiniModucard System")
+		(comment 1 "Wojciech Szafrański")
 		(comment 2 "Designed in poland")
 	)

Commit message: changed numbering to per-sheet
Parts:
- renumbered C2 to C501, U2 to U501
Changed lines of the file:
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@@
 		(dnp no)
 		(fields_autoplaced yes)
-		(property "Reference" "U2"
+		(property "Reference" "U501"
 			(at 139.7 88.9 0)
 			(show_name no)
@@
 			(project "MMS3_hat_templates"
 				(path "/6596548a-44e0-46d8-8624-fd71cf4a3e17/56050d79-5900-47d6-893d-3da0e8bf5810"
-					(reference "U2")
+					(reference "U501")
 					(unit 1)
 				)
@@
 		(dnp no)
 		(fields_autoplaced yes)
-		(property "Reference" "#PWR045"
+		(property "Reference" "#PWR0504"
 			(at 176.53 73.66 0)
 			(hide yes)
@@
 			(project "MMS3_hat_templates"
 				(path "/6596548a-44e0-46d8-8624-fd71cf4a3e17/56050d79-5900-47d6-893d-3da0e8bf5810"
-					(reference "#PWR045")
+					(reference "#PWR0504")
 					(unit 1)
 				)
@@
 		(dnp no)
 		(fields_autoplaced yes)
-		(property "Reference" "#PWR044"
+		(property "Reference" "#PWR0503"
 			(at 176.53 58.42 0)
 			(hide yes)
@@
 			(project "MMS3_hat_templates"
 				(path "/6596548a-44e0-46d8-8624-fd71cf4a3e17/56050d79-5900-47d6-893d-3da0e8bf5810"
-					(reference "#PWR044")
+					(reference "#PWR0503")
 					(unit 1)
 				)
@@
 		(dnp no)
 		(fields_autoplaced yes)
-		(property "Reference" "C2"
+		(property "Reference" "C501"
 			(at 179.07 58.4199 0)
 			(show_name no)
@@
 			(project "MMS3_hat_templates"
 				(path "/6596548a-44e0-46d8-8624-fd71cf4a3e17/56050d79-5900-47d6-893d-3da0e8bf5810"
-					(reference "C2")
+					(reference "C501")
 					(unit 1)
 				)
@@
 		(dnp no)
 		(fields_autoplaced yes)
-		(property "Reference" "#PWR043"
+		(property "Reference" "#PWR0502"
 			(at 154.94 96.52 0)
 			(hide yes)
@@
 			(project "MMS3_hat_templates"
 				(path "/6596548a-44e0-46d8-8624-fd71cf4a3e17/56050d79-5900-47d6-893d-3da0e8bf5810"
-					(reference "#PWR043")
+					(reference "#PWR0502")
 					(unit 1)
 				)
@@
 		(dnp no)
 		(fields_autoplaced yes)
-		(property "Reference" "#PWR042"
+		(property "Reference" "#PWR0501"
 			(at 124.46 113.03 0)
 			(hide yes)
@@
 			(project "MMS3_hat_templates"
 				(path "/6596548a-44e0-46d8-8624-fd71cf4a3e17/56050d79-5900-47d6-893d-3da0e8bf5810"
-					(reference "#PWR042")
+					(reference "#PWR0501")
 					(unit 1)
 				)

Commit message: connected #WC to GND
Connections:
- net GND: now also U501.7 (#WC)
- no-connect marks 1 -> 0
Changed lines of the file:
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@@
 		(color 0 0 0 0)
 	)
-	(no_connect
-		(at 152.4 99.06)
-	)
 	(bus_entry
-		(at 171.45 99.06)
+		(at 186.69 99.06)
 		(size -2.54 2.54)
 		(stroke
@@
 	)
 	(bus_entry
-		(at 171.45 101.6)
+		(at 186.69 101.6)
 		(size -2.54 2.54)
 		(stroke
@@
 		)
 	)
+	(wire
+		(pts
+			(xy 152.4 96.52) (xy 154.94 96.52)
+		)
+		(stroke
+			(width 0)
+			(type default)
+		)
+	)
 	(bus
 		(pts
-			(xy 171.45 99.06) (xy 171.45 101.6)
+			(xy 186.69 99.06) (xy 186.69 101.6)
 		)
 		(stroke
@@
 	(bus
 		(pts
-			(xy 171.45 97.79) (xy 171.45 99.06)
-		)
-		(stroke
-			(width 0)
-			(type default)
-		)
-	)
-	(wire
-		(pts
-			(xy 124.46 99.06) (xy 124.46 96.52)
-		)
-		(stroke
-			(width 0)
-			(type default)
-		)
-	)
-	(wire
-		(pts
-			(xy 152.4 101.6) (xy 168.91 101.6)
+			(xy 186.69 97.79) (xy 186.69 99.06)
 		)
 		(stroke
@@
 	(wire
 		(pts
-			(xy 152.4 96.52) (xy 154.94 96.52)
-		)
-		(stroke
-			(width 0)
-			(type default)
-		)
-	)
-	(wire
-		(pts
-			(xy 152.4 104.14) (xy 168.91 104.14)
+			(xy 124.46 96.52) (xy 124.46 99.06)
 		)
 		(stroke
@@
 	(bus
 		(pts
-			(xy 173.99 97.79) (xy 171.45 97.79)
+			(xy 189.23 97.79) (xy 186.69 97.79)
 		)
 		(stroke
@@
 	(wire
 		(pts
+			(xy 156.21 99.06) (xy 156.21 107.95)
+		)
+		(stroke
+			(width 0)
+			(type default)
+		)
+	)
+	(wire
+		(pts
 			(xy 176.53 54.61) (xy 176.53 57.15)
 		)
@@
 	(wire
 		(pts
+			(xy 152.4 104.14) (xy 184.15 104.14)
+		)
+		(stroke
+			(width 0)
+			(type default)
+		)
+	)
+	(wire
+		(pts
+			(xy 156.21 99.06) (xy 152.4 99.06)
+		)
+		(stroke
+			(width 0)
+			(type default)
+		)
+	)
+	(wire
+		(pts
+			(xy 152.4 101.6) (xy 184.15 101.6)
+		)
+		(stroke
+			(width 0)
+			(type default)
+		)
+	)
+	(wire
+		(pts
 			(xy 124.46 106.68) (xy 124.46 104.14)
 		)
@@
 	)
 	(label "Chainbus.SDA"
-		(at 153.67 104.14 0)
+		(at 168.91 104.14 0)
 		(effects
 			(font
@@
 	)
 	(label "Chainbus.SCL"
-		(at 153.67 101.6 0)
+		(at 168.91 101.6 0)
 		(effects
 			(font
@@
 	(hierarchical_label "Chainbus{I2C}"
 		(shape bidirectional)
-		(at 173.99 97.79 0)
+		(at 189.23 97.79 0)
 		(effects
 			(font
@@
 					(unit 1)
 				)
+			)
+		)
+	)
+	(symbol
+		(lib_id "power:GND")
+		(at 156.21 107.95 0)
+		(unit 1)
+		(body_style 1)
+		(exclude_from_sim no)
+		(in_bom yes)
+		(on_board yes)
+		(in_pos_files yes)
+		(dnp no)
+		(fields_autoplaced yes)
+		(property "Reference" "#PWR0505"
+			(at 156.21 114.3 0)
+			(hide yes)
+			(show_name no)
+			(do_not_autoplace no)
+			(effects
+				(font
+					(size 1.27 1.27)
+				)
+			)
+		)
+		(property "Value" "GND"
+			(at 156.21 113.03 0)
+			(show_name no)
+			(do_not_autoplace no)
+			(effects
+				(font
+					(size 1.27 1.27)
+				)
+			)
+		)
+		(property "Footprint" ""
+			(at 156.21 107.95 0)
+			(hide yes)
+			(show_name no)
+			(do_not_autoplace no)
+			(effects
+				(font
+					(size 1.27 1.27)
+				)
+			)
+		)
+		(property "Datasheet" ""
+			(at 156.21 107.95 0)
+			(hide yes)
+			(show_name no)
+			(do_not_autoplace no)
+			(effects
+				(font
+					(size 1.27 1.27)
+				)
+			)
+		)
+		(property "Description" "Power symbol creates a global label with name \"GND\" , ground"
+			(at 156.21 107.95 0)
+			(hide yes)
+			(show_name no)
+			(do_not_autoplace no)
+			(effects
+				(font
+					(size 1.27 1.27)
+				)
+			)
+		)
+		(pin "1"
+		)
+		(instances
+			(project "MMS3_hat_templates"
+				(path "/6596548a-44e0-46d8-8624-fd71cf4a3e17/56050d79-5900-47d6-893d-3da0e8bf5810"
+					(reference "#PWR0505")
+					(unit 1)
+				)
